Commit message: basic_function_done

File: urdf/robot.xacro (robot description, xacro)
@@ -157,5 +157,5 @@
   <!-- which is correspond to this command <child link="right_camera_link"/> -->
 <!-- sonar -->
-  <xacro:include filename="$(find caracara_gazebo)/urdf/multibeam_sonar_blueview_p900.xacro" />
+  <xacro:include filename="$(find lias_ocean_sim)/urdf/multibeam_sonar_blueview_p900.xacro" />
   <xacro:arg name="standalone" default="false"/>
   <xacro:arg name="gpu_ray" default="false"/>

File: urdf/sensor/camera/camera.xacro (robot description, xacro)
@@ -30,5 +30,5 @@
       mass="0.1"
       update_rate="${update_rate}"
-      hfov="1.5125"
+      hfov="1.5707"
       width="${width}"
       height="${height}"
@@ -37,21 +37,4 @@
       <inertia ixx="0.00001" ixy="0.0" ixz="0.0" iyy="0.00001" iyz="0.0" izz="0.00001" />
       <xacro:insert_block name="origin" />
-    </xacro:regular_camera_plugin_macro>
-  </xacro:macro>
-  <xacro:macro name="wideangle_camera" params="namespace parent_link suffix *origin">
-    <xacro:regular_camera_plugin_macro
-      namespace="${namespace}"
-      suffix="${suffix}"
-      parent_link="${parent_link}"
-      topic="camera"
-      mass="0.015"
-      update_rate="30"
-      hfov="1.8125"
-      width="768"
-      height="492"
-      stddev="0.02"
-      scale="1.0">
-      <inertia ixx="0.00001" ixy="0.0" ixz="0.0" iyy="0.00001" iyz="0.0" izz="0.00001" />
-      <xacro:insert_block name="origin" />>
     </xacro:regular_camera_plugin_macro>
   </xacro:macro>
@@ -105,5 +88,7 @@
         <update_rate>${update_rate}</update_rate>
         <camera name="camera${suffix}">
+          <!--定义水平视野场，1.5125此处为86.7度-->
           <horizontal_fov>${hfov}</horizontal_fov>
+          <!--image标签，功能是定义以像素为单位的图片大小和图片格式-->
           <image>
             <width>${width}</width>
@@ -111,8 +96,10 @@
             <format>R8G8B8</format>
           </image>
+          <!--定义远、近剪裁面，不会渲染远、近剪裁平面之外的对象-->
           <clip>
             <near>0.05</near>
             <far>3000</far>
           </clip>
+          <!--噪音标签，定义噪音模型，它将应用到生成的图片上-->
           <noise>
             <type>gaussian</type>
@@ -125,4 +112,14 @@
           <cameraName>${namespace}/camera${suffix}</cameraName>
           <frameName>camera${suffix}_link_optical</frameName>
+          <CxPrime>${width}/2</CxPrime>
+          <Cx>${width}/2</Cx>
+          <Cy>${height}/2</Cy>
+          <hackBaseline>0</hackBaseline>
+          <focalLength>320.030826</focalLength>
+          <distortionK1>0.0</distortionK1>
+          <distortionK2>0.0</distortionK2>
+          <distortionK3>0.0</distortionK3>
+          <distortionT1>0.0</distortionT1>
+          <distortionT2>0.0</distortionT2>
           <attenuationR>0.0</attenuationR>
           <attenuationG>0.0</attenuationG>
@@ -133,92 +130,8 @@
           <!-- required for ros depth cam -->
           <imageTopicName>${topic}_image</imageTopicName>
-          <pointCloudTopicName>${topic}_cloud</pointCloudTopicName>
+          <cameraInfoTopicName>camera_info</cameraInfoTopicName><!--用于发布相机信息的主题名称为camera_info-->
+          <!-- <pointCloudTopicName>${topic}_cloud</pointCloudTopicName>
           <depthImageTopicName>${topic}_depth</depthImageTopicName>
-          <depthImageCameraInfoTopicName>${topic}_depth_info</depthImageCameraInfoTopicName>
-          <pointCloudCutoff>10.0</pointCloudCutoff>
-        </plugin>
-      </sensor>
-    </gazebo>
-  </xacro:macro>
-  <xacro:macro name="underwater_camera_plugin_macro"
-    params="namespace suffix parent_link topic mass update_rate
-      hfov width height stddev
-      *inertia *origin">
-    <!-- Sensor link -->
-    <link name="${namespace}/camera${suffix}_link">
-      <inertial>
-        <xacro:insert_block name="inertia" />
-        <mass value="${mass}" />
-        <origin xyz="0 0 0" rpy="0 0 0" />
-      </inertial>
-      <visual>
-        <geometry>
-          <mesh filename="file://$(find uuv_sensor_ros_plugins)/meshes/oe14-372.dae" scale="1 1 1"/>
-        </geometry>
-      </visual>
-      <xacro:no_collision/>
-    </link>
-    <joint name="${namespace}/camera${suffix}_joint" type="revolute">
-      <xacro:insert_block name="origin" />
-      <parent link="${parent_link}" />
-      <child link="${namespace}/camera${suffix}_link" />
-      <axis xyz="1 0 0"/>
-      <limit upper="0" lower="0" effort="0" velocity="0" />
-    </joint>
-    <link name="${namespace}/camera${suffix}_link_optical">
-      <xacro:box_inertial x="0.0001" y="0.0001" z="0.0001" mass="0.001">
-        <origin xyz="0 0 0" rpy="0 0 0"/>
-      </xacro:box_inertial>
-      <collision>
-        <!-- todo: gazebo needs a collision volume or it will ignore the pose of
-           the joint that leads to this link (and assume it to be the identity) -->
-        <geometry>
-          <cylinder length="0.000001" radius="0.000001"/>
-        </geometry>
-        <origin xyz="0 0 0" rpy="0 ${0.5*pi} 0"/>
-      </collision>
-    </link>
-    <joint name="${namespace}/camera${suffix}_optical_joint" type="revolute">
-      <origin xyz="0 0 0" rpy="${-pi/2} 0 ${-pi/2}"/>
-      <parent link="${namespace}/camera${suffix}_link"/>
-      <child link="${namespace}/camera${suffix}_link_optical"/>
-      <limit upper="0" lower="0" effort="0" velocity="0" />
-      <axis xyz="1 0 0"/>
-    </joint>
-    <gazebo reference="${namespace}/camera${suffix}_link">
-      <sensor type="depth" name="camera${suffix}">
-        <update_rate>${update_rate}</update_rate>
-        <camera name="camera${suffix}">
-          <horizontal_fov>${hfov}</horizontal_fov>
-          <image>
-            <width>${width}</width>
-            <height>${height}</height>
-            <format>R8G8B8</format>
-          </image>
-          <clip>
-            <near>0.1</near>
-            <far>3000</far>
-          </clip>
-          <noise>
-            <type>gaussian</type>
-            <mean>0.0</mean>
-            <stddev>${stddev}</stddev>
-          </noise>
-        </camera>
-        <plugin name="camera${suffix}_controller" filename="libuuv_gazebo_ros_camera_plugin.so">
-          <updateRate>${update_rate}</updateRate>
-          <cameraName>${namespace}/camera${suffix}</cameraName>
-          <frameName>${namespace}/camera${suffix}_link</frameName>
-          <attenuationR>0.01</attenuationR>
-          <attenuationG>0.01</attenuationG>
-          <attenuationB>0.003</attenuationB>
-          <backgroundR>0</backgroundR>
-          <backgroundG>0</backgroundG>
-          <backgroundB>0</backgroundB>
-          <!-- required for ros depth cam -->
-          <imageTopicName>${topic}_image</imageTopicName>
-          <pointCloudTopicName>${topic}_cloud</pointCloudTopicName>
-          <depthImageTopicName>${topic}_depth</depthImageTopicName>
-          <depthImageCameraInfoTopicName>${topic}_depth_info</depthImageCameraInfoTopicName>
+          <depthImageCameraInfoTopicName>${topic}_depth_info</depthImageCameraInfoTopicName> -->
           <pointCloudCutoff>10.0</pointCloudCutoff>
         </plugin>

File: urdf/sensor/multibeam_sonar_blueview_p900_standalone.xacro (robot description, xacro)
@@ -167,5 +167,5 @@
     </gazebo>
   </xacro:macro>
-  <xacro:macro name="p900_raster_macro"
+  <xacro:macro name="multibeam_blueview_p900_raster_standalone_macro"
                params="name scale sonar_image_topic debug
                sonar_image_raw_topic maxDistance raySkips plotScaler sensorGain writeLog
@@ -186,3 +186,20 @@
     <xacro:multibeam_blueview_p900_visual_ray name="${name}" ray_visual="${ray_visual}" />
   </xacro:macro>
+  <xacro:multibeam_blueview_p900_raster_standalone_macro
+            name="$(arg name)" scale="$(arg scale)" debug="$(arg debug)"
+            sonar_image_topic="$(arg sonar_image_topic)"
+            sonar_image_raw_topic="$(arg sonar_image_raw_topic)"
+            maxDistance="$(arg maxDistance)" raySkips="$(arg raySkips)"
+            plotScaler="$(arg plotScaler)" sensorGain="$(arg sensorGain)"
+            writeLog="$(arg writeLog)" writeFrameInterval="$(arg writeFrameInterval)"
+            artificialVehicleVibration="$(arg artificialVehicleVibration)"
+            constantReflectivity="$(arg constantReflectivity)"
+            reflectivityDatabaseFile="$(arg reflectivityDatabaseFile)"
+            ray_visual="$(arg ray_visual)"/>
+  <xacro:multibeam_sonar_standalone_link name="$(arg name)"/>
+  <joint name="multibeam_sonar_joint" type="fixed">
+    <parent link="$(arg name)_standalone_base_link"/>
+    <child link="$(arg name)_link"/>
+  </joint>
+  <xacro:multibeam_blueview_p900_link name="$(arg name)" scale="$(arg scale)"/>
 </robot>

File: urdf/sensor/rexrov_sensors_main.xacro (robot description, xacro)
@@ -27,5 +27,5 @@
   </xacro:default_imu_macro>
   <!-- Mount cameras -->
-  <xacro:include filename="$(find lias_ocean_sim)/urdf/sensor/camera.xacro" />
+  <xacro:include filename="$(find lias_ocean_sim)/urdf/sensor/camera/camera.xacro" />
   <xacro:camera namespace="${namespace}" parent_link="${namespace}/base_link" suffix="right" update_rate="10" width="640" height="480">
     <origin xyz="1.15 -0.63 0.4" rpy="0 0 0"/>
@@ -43,22 +43,3 @@
     parent_link="${namespace}/base_link"
     inertial_reference_frame="${inertial_reference_frame}" />
-  <!-- sonar -->
-  <xacro:include filename="$(find caracara_gazebo)/urdf/multibeam_sonar_blueview_p900.xacro" />
-  <xacro:multibeam_blueview_p900_raster_standalone_macro
-            name="blueview_p900" scale="1 1 1" debug="false"
-            sonar_image_topic="sonar_image"
-            sonar_image_raw_topic="sonar_image_raw"
-            maxDistance="20" raySkips="10"
-            plotScaler="0" sensorGain="0.02"
-            writeLog="false" writeFrameInterval="5"
-            artificialVehicleVibration="false"
-            constantReflectivity="true"
-            reflectivityDatabaseFile="variationalReflectivityDatabase.csv"
-            ray_visual="true"/>
-  <xacro:multibeam_blueview_p900_link name="$(arg name)" scale="$(arg scale)"/>
-  <joint name="multibeam_sonar_joint" type="fixed">
-    <parent link="${namespace}/base_link"/>
-    <origin xyz="1.2 0 0.2" rpy="0 0 0"/>
-    <child link="$(arg name)_link"/>
-  </joint>
 </robot>
