Commit message: sonar on rexrov function properly

File: urdf/caracara_main.xacro (robot description, xacro)
@@ -157,10 +157,10 @@
   <!-- which is correspond to this command <child link="right_camera_link"/> -->
 <!-- sonar -->
-  <xacro:include filename="$(find lias_ocean_sim)/urdf/multibeam_sonar_blueview_p900.xacro" />
+  <xacro:include filename="$(find lias_ocean_sim)/urdf/sensor/sonar/multibeam_sonar_blueview_p900.xacro" />
   <xacro:arg name="standalone" default="false"/>
   <xacro:arg name="gpu_ray" default="false"/>
   <xacro:arg name="name" default="blueview_p900"/>
   <xacro:arg name="maxDistance" default="10"/>
-  <xacro:arg name="raySkips" default="10"/>
+  <xacro:arg name="raySkips" default="1"/>
   <xacro:arg name="scale" default="1 1 1"/>
   <xacro:arg name="sonar_image_topic" default="sonar_image"/>
@@ -179,5 +179,5 @@
   <xacro:arg name="fidelity" default="500"/>
   <xacro:arg name="robot_name" default=""/>
-  <xacro:multibeam_blueview_p900_raster_standalone_macro
+  <xacro:p900_raster_macro
             name="$(arg name)" scale="$(arg scale)" debug="$(arg debug)"
             sonar_image_topic="$(arg sonar_image_topic)"

File: urdf/sensor/rexrov_sensors_main.xacro (robot description, xacro)
@@ -43,3 +43,22 @@
     parent_link="${namespace}/base_link"
     inertial_reference_frame="${inertial_reference_frame}" />
+  <!-- sonar -->
+  <xacro:include filename="$(find lias_ocean_sim)/urdf/sensor/sonar/multibeam_sonar_blueview_p900.xacro" />
+  <xacro:p900_raster_macro
+            name="blueview_p900" scale="'1 1 1'" debug="false"
+            sonar_image_topic="sonar_image"
+            sonar_image_raw_topic="sonar_image_raw"
+            maxDistance="10" raySkips="1"
+            plotScaler="0" sensorGain="0.02"
+            writeLog="false" writeFrameInterval="5"
+            artificialVehicleVibration="false"
+            constantReflectivity="true"
+            reflectivityDatabaseFile="variationalReflectivityDatabase.csv"
+            ray_visual="true"/>
+  <xacro:multibeam_blueview_p900_link name="$(arg name)" scale="$(arg scale)"/>
+  <joint name="multibeam_sonar_joint" type="fixed">
+    <parent link="${namespace}/base_link"/>
+    <origin xyz="1.2 0 0.2" rpy="0 0 0"/>
+    <child link="$(arg name)_link"/>
+  </joint>
 </robot>
