Commit message: sio_fake

File: urdf/sensor/camera/camera.xacro (robot description, xacro)
@@ -112,9 +112,9 @@
           <cameraName>${namespace}/camera${suffix}</cameraName>
           <frameName>camera${suffix}_link_optical</frameName>
-          <CxPrime>${width}/2</CxPrime>
+          <!-- <CxPrime>${width}/2</CxPrime>
           <Cx>${width}/2</Cx>
-          <Cy>${height}/2</Cy>
+          <Cy>${height}/2</Cy> -->
           <hackBaseline>0</hackBaseline>
-          <focalLength>320.030826</focalLength>
+          <!-- <focalLength>320.030826</focalLength> -->
           <distortionK1>0.0</distortionK1>
           <distortionK2>0.0</distortionK2>

File: urdf/sensor/rexrov_sensors_main.xacro (robot description, xacro)
@@ -9,14 +9,4 @@
     <origin xyz="-1.4 0 -0.312" rpy="0 ${0.5*pi} 0"/>
   </xacro:default_dvl_macro>
-  <!-- Magnetometer  -->
-  <xacro:default_magnetometer namespace="${namespace}" parent_link="${namespace}/base_link"/>
-  <!-- RPT  -->
-  <xacro:default_rpt namespace="${namespace}" parent_link="${namespace}/base_link">
-    <origin xyz="-1.32 0 0.8" rpy="0 0 0"/>
-  </xacro:default_rpt>
-  <!-- Pressure  -->
-  <xacro:default_pressure_macro namespace="${namespace}" parent_link="${namespace}/base_link">
-    <origin xyz="-1.32 0.5 0.85" rpy="0 0 0"/>
-  </xacro:default_pressure_macro>
   <!-- IMU  -->
   <xacro:default_imu_macro
@@ -28,10 +18,9 @@
   <!-- Mount cameras -->
   <xacro:include filename="$(find lias_ocean_sim)/urdf/sensor/camera/camera.xacro" />
-  <xacro:camera namespace="${namespace}" parent_link="${namespace}/base_link" suffix="right" update_rate="10" width="640" height="480">
-    <origin xyz="1.15 -0.63 0.4" rpy="0 0 0"/>
+  <xacro:camera namespace="${namespace}" parent_link="${namespace}/base_link" suffix="right" update_rate="2" width="1920" height="1080">
+    <origin xyz="1.15 -0.2 0.4" rpy="0 0 0"/>
   </xacro:camera>
-  <!-- <xacro:default_camera namespace="${namespace}" parent_link="${namespace}/base_link" suffix="left" update_rate="10" width="768" height="492"> -->
-  <xacro:camera namespace="${namespace}" parent_link="${namespace}/base_link" suffix="left" update_rate="10" width="640" height="480">
-    <origin xyz="1.15 0.63 0.4" rpy="0 0 0"/>
+  <xacro:camera namespace="${namespace}" parent_link="${namespace}/base_link" suffix="left" update_rate="2" width="1920" height="1080">
+    <origin xyz="1.15 0.2 0.4" rpy="0 0 0"/>
   </xacro:camera>
   <!-- <xacro:default_camera namespace="${namespace}" parent_link="${namespace}/base_link" suffix="left"> -->
@@ -45,20 +34,23 @@
   <!-- sonar -->
   <xacro:include filename="$(find lias_ocean_sim)/urdf/sensor/sonar/multibeam_sonar_blueview_p900.xacro" />
-  <xacro:p900_raster_macro
-            name="blueview_p900" scale="'1 1 1'" debug="false"
-            sonar_image_topic="sonar_image"
-            sonar_image_raw_topic="sonar_image_raw"
-            maxDistance="10" raySkips="1"
-            plotScaler="0" sensorGain="0.02"
-            writeLog="false" writeFrameInterval="5"
-            artificialVehicleVibration="false"
-            constantReflectivity="true"
-            reflectivityDatabaseFile="variationalReflectivityDatabase.csv"
-            ray_visual="true"/>
-  <xacro:multibeam_blueview_p900_link name="$(arg name)" scale="$(arg scale)"/>
-  <joint name="multibeam_sonar_joint" type="fixed">
-    <parent link="${namespace}/base_link"/>
+  <xacro:multibeam_blueview_p900_ray_macro
+    name="blueview_p900"
+    scale="1 1 1"
+    debug="false"
+    sonar_image_topic="sonar_image"
+    sonar_image_raw_topic="sonar_image_raw"
+    robot_name="rexrov"
+    maxDistance="20"
+    raySkips="1"
+    plotScaler="0"
+    sensorGain="0.02"
+    writeLog="false"
+    writeFrameInterval="5"
+    gaussian_noise_mean="0。0"
+    gaussian_noise_stddev="0.0"
+    fidelity="500"
+    robot_link="${namespace}/base_link"
+    ray_visual="true">
     <origin xyz="1.2 0 0.2" rpy="0 0 0"/>
-    <child link="$(arg name)_link"/>
-  </joint>
+  </xacro:multibeam_blueview_p900_ray_macro>
 </robot>

File: urdf/sensor/sonar/multibeam_sonar_blueview_p900.xacro (robot description, xacro)
@@ -87,4 +87,82 @@
     </gazebo>
   </xacro:macro>
+  <xacro:macro name="multibeam_blueview_p900_ray_sensor"
+               params="name pcl_topic_name sensor_link sonar_image_topic sonar_image_raw_topic
+               maxDistance raySkips plotScaler sensorGain writeLog writeFrameInterval
+               gaussian_noise_mean gaussian_noise_stddev fidelity debug">
+    <gazebo reference="${sensor_link}">
+      <sensor name="${name}_sensor" type="gpu_ray">
+        <visualize>false</visualize>
+        <always_on>true</always_on>
+        <update_rate>5</update_rate>
+        <ray>
+          <scan>
+            <!-- Set horizontal FOV by setting image height -->
+            <!-- 512 beams with 90 degrees horizontal FOV (M900-90) -->
+            <horizontal>
+              <samples>512</samples>
+              <resolution>1</resolution>
+              <min_angle>-0.78539816339</min_angle>
+              <max_angle>0.78539816339</max_angle>
+            </horizontal>
+            <!-- Set vertical FOV by setting image height -->
+            <!-- Approx 2 times the spec sheet (sepc: 20 deg.) -->
+            <vertical>
+              <samples>${fidelity}</samples>
+              <resolution>1</resolution>
+              <min_angle>-0.349066</min_angle>
+              <max_angle>0.349066</max_angle>
+            </vertical>
+          </scan>
+          <range>
+            <!-- min range is a collision range no need to change-->
+            <min>0.1</min>
+            <max>${maxDistance + 2}</max>
+            <resolution>0.1</resolution>
+          </range>
+          <noise>
+            <type>gaussian</type>
+            <!-- Noise parameters based on published spec for Hokuyo laser
+                achieving "+-30mm" accuracy at range < 10m.  A mean of 0.0m and
+                stddev of 0.01m will put 99.7% of samples within 0.03m of the true
+                reading. -->
+            <mean>${gaussian_noise_mean}</mean>
+            <stddev>${gaussian_noise_stddev}</stddev>
+          </noise>
+        </ray>
+        <plugin name="${name}_ray_sonar_sensor" filename="libgazebo_ros_velodyne_gpu_laser.so">
+           <topicName>${name}_point_cloud</topicName>
+           <!-- <frameName>${name}_forward_sonar_optical_link</frameName> -->
+           <organize_cloud>true</organize_cloud>
+           <min_range>0.2</min_range>
+           <max_range>${maxDistance}</max_range>
+        </plugin>
+        <plugin filename="libnps_multibeam_sonar_ray_ros_plugin.so" name="${name}_sensor_controller">
+          <!-- Sonar properties -->
+          <verticalFOV>20</verticalFOV>
+          <sonarFreq>900e3</sonarFreq>
+          <bandwidth>29.9e3</bandwidth>
+          <soundSpeed>1500</soundSpeed>
+          <sourceLevel>220</sourceLevel>
+          <maxDistance>${maxDistance}</maxDistance>
+          <raySkips>${raySkips}</raySkips>
+          <sensorGain>${sensorGain}</sensorGain>
+          <plotScaler>${plotScaler}</plotScaler>
+          <writeLog>${writeLog}</writeLog>
+          <debugFlag>${debug}</debugFlag>
+          <writeFrameInterval>${writeFrameInterval}</writeFrameInterval>
+          <!-- This name is prepended to ROS topics -->
+          <cameraName>${name}</cameraName>
+          <!-- ROS publication topics -->
+          <imageTopicName>image_raw</imageTopicName>
+          <cameraInfoTopicName>image_raw/camera_info</cameraInfoTopicName>
+          <pointCloudTopicName>${pcl_topic_name}</pointCloudTopicName>
+          <sonarImageRawTopicName>${sonar_image_raw_topic}</sonarImageRawTopicName>
+          <sonarImageTopicName>${sonar_image_topic}</sonarImageTopicName>
+          <frameName>${name}_forward_sonar_optical_link</frameName>
+        </plugin>
+      </sensor>
+    </gazebo>
+  </xacro:macro>
   <xacro:macro name="multibeam_sonar_visual_link" params="name">
     <link name="${name}_visual_ray_link">
@@ -160,4 +238,94 @@
        but sensor orientation will always be forward and down relative to
        the robot link (robot_link parameter). -->
+  <xacro:macro name="multibeam_blueview_p900_raster_macro"
+               params="name scale sonar_image_topic debug
+               sonar_image_raw_topic maxDistance raySkips plotScaler sensorGain writeLog
+               writeFrameInterval artificialVehicleVibration constantReflectivity
+               reflectivityDatabaseFile robot_link ray_visual">
+    <xacro:multibeam_blueview_p900_link name="${name}" scale="${scale}"/>
+    <joint name="multibeam_sonar_joint" type="fixed">
+      <parent link="${robot_link}"/>
+      <child link="${name}_link"/>
+      <xacro:insert_block name="origin"/>\
+    </joint>
+    <xacro:multibeam_blueview_p900_raster_sensor name="${name}" debug="${debug}"
+                               sonar_image_topic="${sonar_image_topic}"  sensor_link="${name}_link"
+                               sonar_image_raw_topic="${sonar_image_raw_topic}"
+                               maxDistance="${maxDistance}" raySkips="${raySkips}"
+                               plotScaler="${plotScaler}" sensorGain="${sensorGain}"
+                               writeLog="${writeLog}" writeFrameInterval="${writeFrameInterval}"
+                               artificialVehicleVibration="${artificialVehicleVibration}"
+                               constantReflectivity="${constantReflectivity}"
+                               reflectivityDatabaseFile="${reflectivityDatabaseFile}"/>
+    <!-- Ray Visual -->
+    <xacro:multibeam_sonar_visual_link name="${name}"/>
+    <xacro:multibeam_sonar_visual_joint name="${name}"/>
+    <xacro:multibeam_blueview_p900_visual_ray name="${name}" ray_visual="${ray_visual}"/>
+  </xacro:macro>
+  <xacro:macro name="multibeam_blueview_p900_ray_macro"
+               params="name scale debug sonar_image_topic sonar_image_raw_topic
+               robot_name
+               maxDistance raySkips plotScaler sensorGain writeLog
+               writeFrameInterval gaussian_noise_mean gaussian_noise_stddev fidelity
+               robot_link ray_visual *origin">
+    <xacro:multibeam_blueview_p900_link name="${name}" scale="${scale}"/>
+    <joint name="multibeam_sonar_joint" type="fixed">
+      <parent link="${robot_link}"/>
+      <child link="${name}_link"/>
+      <xacro:insert_block name="origin"/>\
+    </joint>
+    <xacro:multibeam_blueview_p900_ray_sensor name="${name}" sensor_link="${name}_link"
+                               sonar_image_topic="${sonar_image_topic}" debug="${debug}"
+                               sonar_image_raw_topic="${sonar_image_raw_topic}"
+                               maxDistance="${maxDistance}" raySkips="${raySkips}"
+                               plotScaler="${plotScaler}" sensorGain="${sensorGain}"
+                               writeLog="${writeLog}" writeFrameInterval="${writeFrameInterval}"
+                               gaussian_noise_mean="${gaussian_noise_mean}"
+                               gaussian_noise_stddev="${gaussian_noise_stddev}"
+                               fidelity="${fidelity}" pcl_topic_name="${robot_name}/${name}_point_cloud"/>
+    <!-- Ray Visual -->
+    <xacro:multibeam_sonar_visual_link name="${name}"/>
+    <xacro:multibeam_sonar_visual_joint name="${name}"/>
+    <xacro:multibeam_blueview_p900_visual_ray name="${name}" ray_visual="${ray_visual}"/>
+  </xacro:macro>
+  <xacro:macro name="multibeam_blueview_p900_macro"
+               params="name scale sonar_image_topic debug gpu_ray robot_name
+               sonar_image_raw_topic maxDistance raySkips plotScaler sensorGain writeLog
+               writeFrameInterval gaussian_noise_mean gaussian_noise_stddev fidelity
+               artificialVehicleVibration constantReflectivity reflectivityDatabaseFile
+               robot_link ray_visual *origin">
+    <xacro:multibeam_blueview_p900_link name="${name}" scale="${scale}"/>
+    <joint name="multibeam_sonar_joint" type="fixed">
+      <parent link="${robot_link}"/>
+      <child link="${name}_link"/>
+      <xacro:insert_block name="origin"/>
+    </joint>
+    <xacro:if value="$(arg gpu_ray)">
+      <xacro:multibeam_blueview_p900_ray_sensor name="${name}" sensor_link="${name}_link"
+                                sonar_image_topic="${sonar_image_topic}" debug="${debug}"
+                                sonar_image_raw_topic="${sonar_image_raw_topic}"
+                                maxDistance="${maxDistance}" raySkips="${raySkips}"
+                                plotScaler="${plotScaler}" sensorGain="${sensorGain}"
+                                writeLog="${writeLog}" writeFrameInterval="${writeFrameInterval}"
+                                gaussian_noise_mean="${gaussian_noise_mean}"
+                                gaussian_noise_stddev="${gaussian_noise_stddev}"
+                                fidelity="${fidelity}" pcl_topic_name="${robot_name}/${name}_point_cloud"/>
+    </xacro:if>
+    <xacro:unless value="$(arg gpu_ray)">
+      <xacro:multibeam_blueview_p900_raster_sensor name="${name}" debug="${debug}"
+                                sonar_image_topic="${sonar_image_topic}"  sensor_link="${name}_link"
+                                sonar_image_raw_topic="${sonar_image_raw_topic}"
+                                maxDistance="${maxDistance}" raySkips="${raySkips}"
+                                plotScaler="${plotScaler}" sensorGain="${sensorGain}"
+                                writeLog="${writeLog}" writeFrameInterval="${writeFrameInterval}"
+                                artificialVehicleVibration="${artificialVehicleVibration}"
+                                constantReflectivity="${constantReflectivity}"
+                                reflectivityDatabaseFile="${reflectivityDatabaseFile}"/>
+    </xacro:unless>
+    <!-- Ray Visual -->
+    <xacro:multibeam_sonar_visual_link name="${name}"/>
+    <xacro:multibeam_sonar_visual_joint name="${name}"/>
+    <xacro:multibeam_blueview_p900_visual_ray name="${name}" ray_visual="${ray_visual}"/>
+  </xacro:macro>
   <!-- For standalone -->
   <xacro:macro name="multibeam_sonar_standalone_link" params="name">
@@ -167,9 +335,15 @@
     </gazebo>
   </xacro:macro>
-  <xacro:macro name="p900_raster_macro"
+  <xacro:macro name="multibeam_blueview_p900_raster_standalone_macro"
                params="name scale sonar_image_topic debug
                sonar_image_raw_topic maxDistance raySkips plotScaler sensorGain writeLog
                writeFrameInterval artificialVehicleVibration constantReflectivity
                reflectivityDatabaseFile ray_visual">
+    <xacro:multibeam_sonar_standalone_link name="${name}"/>
+    <xacro:multibeam_blueview_p900_link name="${name}" scale="${scale}"/>
+    <joint name="multibeam_sonar_joint" type="fixed">
+      <parent link="${name}_standalone_base_link"/>
+      <child link="${name}_link"/>
+    </joint>
     <xacro:multibeam_blueview_p900_raster_sensor name="${name}" sensor_link="${name}_link"
                                sonar_image_topic="${sonar_image_topic}"  debug="${debug}"
@@ -186,3 +360,55 @@
     <xacro:multibeam_blueview_p900_visual_ray name="${name}" ray_visual="${ray_visual}" />
   </xacro:macro>
+  <xacro:macro name="multibeam_blueview_p900_ray_standalone_macro"
+               params="name scale sonar_image_topic fidelity debug robot_name
+               sonar_image_raw_topic maxDistance raySkips plotScaler sensorGain writeLog
+               writeFrameInterval gaussian_noise_mean gaussian_noise_stddev ray_visual">
+    <xacro:multibeam_sonar_standalone_link name="${name}"/>
+    <xacro:multibeam_blueview_p900_link name="${name}" scale="${scale}"/>
+    <joint name="multibeam_sonar_joint" type="fixed">
+      <parent link="${name}_standalone_base_link"/>
+      <child link="${name}_link"/>
+    </joint>
+    <xacro:multibeam_blueview_p900_ray_sensor name="${name}" sensor_link="${name}_link"
+                               sonar_image_topic="${sonar_image_topic}"  debug="${debug}"
+                               sonar_image_raw_topic="${sonar_image_raw_topic}"
+                               maxDistance="${maxDistance}" raySkips="${raySkips}"
+                               plotScaler="${plotScaler}" sensorGain="${sensorGain}"
+                               writeLog="${writeLog}" writeFrameInterval="${writeFrameInterval}"
+                               gaussian_noise_mean="${gaussian_noise_mean}"
+                               gaussian_noise_stddev="${gaussian_noise_stddev}"
+                               fidelity="${fidelity}" pcl_topic_name="${name}_point_cloud"/>
+    <!-- Ray Visual -->
+    <xacro:multibeam_sonar_visual_link name="${name}"/>
+    <xacro:multibeam_sonar_visual_joint name="${name}"/>
+    <xacro:multibeam_blueview_p900_visual_ray name="${name}" ray_visual="${ray_visual}" />
+  </xacro:macro>
+  <xacro:if value="$(arg standalone)">
+    <xacro:unless value="$(arg gpu_ray)">
+      <xacro:multibeam_blueview_p900_raster_standalone_macro
+                name="$(arg name)" scale="$(arg scale)" debug="$(arg debug)"
+                sonar_image_topic="$(arg sonar_image_topic)"
+                sonar_image_raw_topic="$(arg sonar_image_raw_topic)"
+                maxDistance="$(arg maxDistance)" raySkips="$(arg raySkips)"
+                plotScaler="$(arg plotScaler)" sensorGain="$(arg sensorGain)"
+                writeLog="$(arg writeLog)" writeFrameInterval="$(arg writeFrameInterval)"
+                artificialVehicleVibration="$(arg artificialVehicleVibration)"
+                constantReflectivity="$(arg constantReflectivity)"
+                reflectivityDatabaseFile="$(arg reflectivityDatabaseFile)"
+                ray_visual="$(arg ray_visual)"/>
+    </xacro:unless>
+    <xacro:if value="$(arg gpu_ray)">
+      <xacro:multibeam_blueview_p900_ray_standalone_macro
+                name="$(arg name)" scale="$(arg scale)" debug="$(arg debug)"
+                sonar_image_topic="$(arg sonar_image_topic)"
+                sonar_image_raw_topic="$(arg sonar_image_raw_topic)"
+                maxDistance="$(arg maxDistance)" raySkips="$(arg raySkips)"
+                plotScaler="$(arg plotScaler)" sensorGain="$(arg sensorGain)"
+                writeLog="$(arg writeLog)" writeFrameInterval="$(arg writeFrameInterval)"
+                gaussian_noise_mean="$(arg gaussian_noise_mean)"
+                gaussian_noise_stddev="$(arg gaussian_noise_stddev)"
+                fidelity="$(arg fidelity)" robot_name=""
+                ray_visual="$(arg ray_visual)"/>
+    </xacro:if>
+  </xacro:if>
 </robot>
