Commit message: charuco done

File: urdf/sensor/camera/camera.xacro (robot description, xacro)
@@ -30,5 +30,5 @@
       mass="0.1"
       update_rate="${update_rate}"
-      hfov="1.5707"
+      hfov="0.785"
       width="${width}"
       height="${height}"
@@ -99,5 +99,5 @@
           <clip>
             <near>0.05</near>
-            <far>3000</far>
+            <far>50</far>
           </clip>
           <!--噪音标签，定义噪音模型，它将应用到生成的图片上-->

File: urdf/sensor/rexrov_sensors_main.xacro (robot description, xacro)
@@ -1,13 +1,35 @@
 <?xml version="1.0"?>
 <!-- Note the detailed sensor configuration can be found in $(find uuv_sensor_ros_plugins)/urdf/-->
+<!-- cd ~/catkin_ws/src/uuv_simulator/uuv_sensor_plugins/uuv_sensor_ros_plugins/urdf$  -->
+<!-- Please modify the default_dvl_macro in dvl_snippets.xacro -->
+  <!-- <xacro:macro name="default_dvl_macro" params="namespace parent_link *origin inertial_reference_frame">
+    <xacro:dvl_plugin_macro
+      namespace="${namespace}"
+      suffix=""
+      parent_link="${parent_link}"
+      reference_frame="${inertial_reference_frame}"
+      update_rate="${update_rate}"
+      topic="dvl"
+      noise_sigma="${noise_sigma}"
+      noise_amplitude="${noise_amplitude}"
+      scale="1">
+      <xacro:insert_block name="origin" />
+    </xacro:dvl_plugin_macro>
+  </xacro:macro> -->
 <robot xmlns:xacro="http://www.ros.org/wiki/xacro">
   <!-- DVL  -->
+  <!-- 典型的DVL更新率在4-15Hz之间 -->
+  <!-- 实际数据显示协方差约为3.79e-05，所以噪声标准差≈sqrt(3.79e-05)=0.006 -->
+  <!-- 噪声振幅，影响测量波动范围,通常设置为noise_sigma的2-3倍 -->
   <xacro:default_dvl_macro
     namespace="${namespace}"
     parent_link="${namespace}/base_link"
+    update_rate="20.0"
+    noise_sigma="0.006"
+    noise_amplitude="0.018"
     inertial_reference_frame="${inertial_reference_frame}">
-    <origin xyz="-1.4 0 -0.312" rpy="0 ${0.5*pi} 0"/>
+    <origin xyz="-1 0 -0.8" rpy="0 ${0.5*pi} 0"/>
   </xacro:default_dvl_macro>
-  <!-- IMU  -->
+  <!-- IMU  50 Hz -->
   <xacro:default_imu_macro
     namespace="${namespace}"
@@ -18,14 +40,14 @@
   <!-- Mount cameras -->
   <xacro:include filename="$(find lias_ocean_sim)/urdf/sensor/camera/camera.xacro" />
-  <xacro:camera namespace="${namespace}" parent_link="${namespace}/base_link" suffix="right" update_rate="2" width="1920" height="1080">
-    <origin xyz="1.15 -0.2 0.4" rpy="0 0 0"/>
+  <xacro:camera namespace="${namespace}" parent_link="${namespace}/base_link" suffix="right" update_rate="20" width="640" height="480">
+    <origin xyz="1.15 0.2 0.4" rpy="0 0.4 0"/>
   </xacro:camera>
-  <xacro:camera namespace="${namespace}" parent_link="${namespace}/base_link" suffix="left" update_rate="2" width="1920" height="1080">
-    <origin xyz="1.15 0.2 0.4" rpy="0 0 0"/>
-  </xacro:camera>
+  <!-- <xacro:camera namespace="${namespace}" parent_link="${namespace}/base_link" suffix="left" update_rate="24" width="640" height="360">
+    <origin xyz="1.15 0.2 0.4" rpy="0 0.4 0"/>
+  </xacro:camera> -->
   <!-- <xacro:default_camera namespace="${namespace}" parent_link="${namespace}/base_link" suffix="left"> -->
   <!-- Mount a GPS. -->
-  <xacro:default_gps namespace="${namespace}" parent_link="${namespace}/base_link" />
-  <!-- Mount a Pose 3D sensor. -->
+  <!-- <xacro:default_gps namespace="${namespace}" parent_link="${namespace}/base_link" /> -->
+  <!-- Mount a Pose 3D sensor. REALLY REALLY important for the controller!!! -->
   <xacro:default_pose_3d_macro
     namespace="${namespace}"
@@ -33,6 +55,6 @@
     inertial_reference_frame="${inertial_reference_frame}" />
   <!-- sonar -->
-  <xacro:include filename="$(find lias_ocean_sim)/urdf/sensor/sonar/multibeam_sonar_blueview_p900.xacro" />
-  <xacro:multibeam_blueview_p900_ray_macro
+  <!-- <xacro:include filename="$(find lias_ocean_sim)/urdf/sensor/sonar/multibeam_sonar_blueview_p900.xacro" />
+  <xacro:sonar_visualization_macro_no_blue_ray
     name="blueview_p900"
     scale="1 1 1"
@@ -41,5 +63,5 @@
     sonar_image_raw_topic="sonar_image_raw"
     robot_name="rexrov"
-    maxDistance="20"
+    maxDistance="10"
     raySkips="1"
     plotScaler="0"
@@ -47,10 +69,30 @@
     writeLog="false"
     writeFrameInterval="5"
-    gaussian_noise_mean="0。0"
+    gaussian_noise_mean="0.0"
     gaussian_noise_stddev="0.0"
     fidelity="500"
     robot_link="${namespace}/base_link"
     ray_visual="true">
-    <origin xyz="1.2 0 0.2" rpy="0 0 0"/>
-  </xacro:multibeam_blueview_p900_ray_macro>
+    <origin xyz="1.2 0 -0.65" rpy="0 0 0"/>
+  </xacro:sonar_visualization_macro_no_blue_ray> -->
+  <!-- <xacro:sonar_visualization_macro
+    name="blueview_p900"
+    scale="1 1 1"
+    debug="false"
+    sonar_image_topic="sonar_image"
+    sonar_image_raw_topic="sonar_image_raw"
+    robot_name="rexrov"
+    maxDistance="10"
+    raySkips="1"
+    plotScaler="0"
+    sensorGain="0.02"
+    writeLog="false"
+    writeFrameInterval="5"
+    gaussian_noise_mean="0.0"
+    gaussian_noise_stddev="0.0"
+    fidelity="500"
+    robot_link="${namespace}/base_link"
+    ray_visual="true">
+    <origin xyz="1.2 0 -0.65" rpy="0 0 0"/>
+  </xacro:sonar_visualization_macro> -->
 </robot>

File: urdf/sensor/sonar/multibeam_sonar_blueview_p900 copy.xacro (robot description, xacro)
@@ -23,4 +23,68 @@
     </link>
   </xacro:macro>
+  <!-- Generates a sensor element with Blueview P900 parameters -->
+  <xacro:macro name="multibeam_blueview_p900_raster_sensor"
+               params="name sensor_link sonar_image_topic sonar_image_raw_topic debug
+               maxDistance raySkips plotScaler sensorGain writeLog writeFrameInterval
+              artificialVehicleVibration constantReflectivity reflectivityDatabaseFile">
+    <gazebo reference="${sensor_link}">
+      <sensor name="${name}_sensor" type="depth">
+        <visualize>true</visualize>
+        <always_on>true</always_on>
+        <update_rate>10</update_rate>
+        <camera>
+          <!-- 90 degrees for the M900-90 -->
+          <horizontal_fov>1.57079632679</horizontal_fov>
+          <image>
+            <width>512</width>
+            <!-- Set vertical FOV by setting image height -->
+            <!-- Approx 2 times the spec sheet (sepc: 20 deg.) -->
+            <height>228</height>
+            <format>R8G8B8</format>
+          </image>
+          <clip>
+            <near>0.2</near>            <!-- optimal 2m-60m -->
+            <far>${maxDistance + 2}</far>
+          </clip>
+          <depth_camera>
+            <output>${name}_depths</output>
+          </depth_camera>
+          <!-- <save enabled="true">
+            <path>/tmp/camera</path>
+          </save> -->
+        </camera>
+        <plugin filename="libnps_multibeam_sonar_ros_plugin.so" name="${name}_sensor_controller">
+          <!-- Sonar properties -->
+          <verticalFOV>20</verticalFOV>
+          <sonarFreq>900e3</sonarFreq>
+          <bandwidth>29.9e3</bandwidth>
+          <soundSpeed>1500</soundSpeed>
+          <sourceLevel>220</sourceLevel>
+          <maxDistance>${maxDistance}</maxDistance>
+          <constantReflectivity>${constantReflectivity}</constantReflectivity>
+          <!-- The CSV databsefile is located at the worlds folder -->
+          <reflectivityDatabaseFile>${reflectivityDatabaseFile}</reflectivityDatabaseFile>
+          <raySkips>${raySkips}</raySkips>
+          <sensorGain>${sensorGain}</sensorGain>
+          <plotScaler>${plotScaler}</plotScaler>
+          <writeLog>${writeLog}</writeLog>
+          <debugFlag>${debug}</debugFlag>
+          <writeFrameInterval>${writeFrameInterval}</writeFrameInterval>
+          <artificialVehicleVibration>${artificialVehicleVibration}</artificialVehicleVibration>
+          <!-- This name is prepended to ROS topics -->
+          <cameraName>${name}</cameraName>
+          <!-- ROS publication topics -->
+          <imageTopicName>${name}/image_raw</imageTopicName>
+          <cameraInfoTopicName>${name}/image_raw/camera_info</cameraInfoTopicName>
+          <pointCloudTopicName>${name}/point_cloud</pointCloudTopicName>
+          <depthImageTopicName>${name}/image_depth</depthImageTopicName>
+          <depthImageCameraInfoTopicName>${name}/image_depth/camera_info</depthImageCameraInfoTopicName>
+          <sonarImageRawTopicName>${sonar_image_raw_topic}</sonarImageRawTopicName>
+          <sonarImageTopicName>${sonar_image_topic}</sonarImageTopicName>
+          <frameName>${name}_forward_sonar_optical_link</frameName>
+        </plugin>
+      </sensor>
+    </gazebo>
+  </xacro:macro>
   <xacro:macro name="multibeam_blueview_p900_ray_sensor"
                params="name pcl_topic_name sensor_link sonar_image_topic sonar_image_raw_topic
@@ -39,14 +103,14 @@
               <samples>512</samples>
               <resolution>1</resolution>
-              <min_angle>-0.52</min_angle>
-              <max_angle>0.52</max_angle>
+              <min_angle>-0.78539816339</min_angle>
+              <max_angle>0.78539816339</max_angle>
             </horizontal>
             <!-- Set vertical FOV by setting image height -->
             <!-- Approx 2 times the spec sheet (sepc: 20 deg.) -->
             <vertical>
-              <samples>512</samples>
+              <samples>${fidelity}</samples>
               <resolution>1</resolution>
-              <min_angle>-0.179066</min_angle>
-              <max_angle>0.179066</max_angle>
+              <min_angle>-0.349066</min_angle>
+              <max_angle>0.349066</max_angle>
             </vertical>
           </scan>
@@ -54,5 +118,5 @@
             <!-- min range is a collision range no need to change-->
             <min>0.1</min>
-            <max>8</max>
+            <max>${maxDistance + 2}</max>
             <resolution>0.1</resolution>
           </range>
@@ -129,6 +193,6 @@
               <samples>100</samples>
               <resolution>1</resolution>
-              <min_angle>-0.52</min_angle>
-              <max_angle>0.52</max_angle>
+              <min_angle>-0.785398</min_angle>
+              <max_angle>0.785398</max_angle>
             </horizontal>
             <vertical>
@@ -167,5 +231,5 @@
   <xacro:arg name="gaussian_noise_mean" default="0.0"/>
   <xacro:arg name="gaussian_noise_stddev" default="0.0"/>
-  <xacro:arg name="fidelity" default="64"/>
+  <xacro:arg name="fidelity" default="500"/>
   <xacro:arg name="robot_name" default=""/>
   <!-- Top level macro for generating the link, sensor, joint combo
@@ -174,4 +238,29 @@
        but sensor orientation will always be forward and down relative to
        the robot link (robot_link parameter). -->
+  <xacro:macro name="multibeam_blueview_p900_raster_macro"
+               params="name scale sonar_image_topic debug
+               sonar_image_raw_topic maxDistance raySkips plotScaler sensorGain writeLog
+               writeFrameInterval artificialVehicleVibration constantReflectivity
+               reflectivityDatabaseFile robot_link ray_visual">
+    <xacro:multibeam_blueview_p900_link name="${name}" scale="${scale}"/>
+    <joint name="multibeam_sonar_joint" type="fixed">
+      <parent link="${robot_link}"/>
+      <child link="${name}_link"/>
+      <xacro:insert_block name="origin"/>\
+    </joint>
+    <xacro:multibeam_blueview_p900_raster_sensor name="${name}" debug="${debug}"
+                               sonar_image_topic="${sonar_image_topic}"  sensor_link="${name}_link"
+                               sonar_image_raw_topic="${sonar_image_raw_topic}"
+                               maxDistance="${maxDistance}" raySkips="${raySkips}"
+                               plotScaler="${plotScaler}" sensorGain="${sensorGain}"
+                               writeLog="${writeLog}" writeFrameInterval="${writeFrameInterval}"
+                               artificialVehicleVibration="${artificialVehicleVibration}"
+                               constantReflectivity="${constantReflectivity}"
+                               reflectivityDatabaseFile="${reflectivityDatabaseFile}"/>
+    <!-- Ray Visual -->
+    <xacro:multibeam_sonar_visual_link name="${name}"/>
+    <xacro:multibeam_sonar_visual_joint name="${name}"/>
+    <xacro:multibeam_blueview_p900_visual_ray name="${name}" ray_visual="${ray_visual}"/>
+  </xacro:macro>
   <xacro:macro name="multibeam_blueview_p900_ray_macro"
                params="name scale debug sonar_image_topic sonar_image_raw_topic
@@ -200,9 +289,9 @@
     <xacro:multibeam_blueview_p900_visual_ray name="${name}" ray_visual="${ray_visual}"/>
   </xacro:macro>
-  <xacro:macro name="sonar_visualization_macro"
-               params="name scale debug sonar_image_topic sonar_image_raw_topic
-               robot_name
-               maxDistance raySkips plotScaler sensorGain writeLog
+  <xacro:macro name="multibeam_blueview_p900_macro"
+               params="name scale sonar_image_topic debug gpu_ray robot_name
+               sonar_image_raw_topic maxDistance raySkips plotScaler sensorGain writeLog
                writeFrameInterval gaussian_noise_mean gaussian_noise_stddev fidelity
+               artificialVehicleVibration constantReflectivity reflectivityDatabaseFile
                robot_link ray_visual *origin">
     <xacro:multibeam_blueview_p900_link name="${name}" scale="${scale}"/>
@@ -210,23 +299,32 @@
       <parent link="${robot_link}"/>
       <child link="${name}_link"/>
-      <xacro:insert_block name="origin"/>\
-    </joint>
+      <xacro:insert_block name="origin"/>
+    </joint>
+    <xacro:if value="$(arg gpu_ray)">
+      <xacro:multibeam_blueview_p900_ray_sensor name="${name}" sensor_link="${name}_link"
+                                sonar_image_topic="${sonar_image_topic}" debug="${debug}"
+                                sonar_image_raw_topic="${sonar_image_raw_topic}"
+                                maxDistance="${maxDistance}" raySkips="${raySkips}"
+                                plotScaler="${plotScaler}" sensorGain="${sensorGain}"
+                                writeLog="${writeLog}" writeFrameInterval="${writeFrameInterval}"
+                                gaussian_noise_mean="${gaussian_noise_mean}"
+                                gaussian_noise_stddev="${gaussian_noise_stddev}"
+                                fidelity="${fidelity}" pcl_topic_name="${robot_name}/${name}_point_cloud"/>
+    </xacro:if>
+    <xacro:unless value="$(arg gpu_ray)">
+      <xacro:multibeam_blueview_p900_raster_sensor name="${name}" debug="${debug}"
+                                sonar_image_topic="${sonar_image_topic}"  sensor_link="${name}_link"
+                                sonar_image_raw_topic="${sonar_image_raw_topic}"
+                                maxDistance="${maxDistance}" raySkips="${raySkips}"
+                                plotScaler="${plotScaler}" sensorGain="${sensorGain}"
+                                writeLog="${writeLog}" writeFrameInterval="${writeFrameInterval}"
+                                artificialVehicleVibration="${artificialVehicleVibration}"
+                                constantReflectivity="${constantReflectivity}"
+                                reflectivityDatabaseFile="${reflectivityDatabaseFile}"/>
+    </xacro:unless>
     <!-- Ray Visual -->
     <xacro:multibeam_sonar_visual_link name="${name}"/>
     <xacro:multibeam_sonar_visual_joint name="${name}"/>
     <xacro:multibeam_blueview_p900_visual_ray name="${name}" ray_visual="${ray_visual}"/>
-  </xacro:macro>
-  <xacro:macro name="sonar_visualization_macro_no_blue_ray"
-               params="name scale debug sonar_image_topic sonar_image_raw_topic
-               robot_name
-               maxDistance raySkips plotScaler sensorGain writeLog
-               writeFrameInterval gaussian_noise_mean gaussian_noise_stddev fidelity
-               robot_link ray_visual *origin">
-    <xacro:multibeam_blueview_p900_link name="${name}" scale="${scale}"/>
-    <joint name="multibeam_sonar_joint" type="fixed">
-      <parent link="${robot_link}"/>
-      <child link="${name}_link"/>
-      <xacro:insert_block name="origin"/>\
-    </joint>
   </xacro:macro>
   <!-- For standalone -->
@@ -236,4 +334,29 @@
       <static>true</static>
     </gazebo>
+  </xacro:macro>
+  <xacro:macro name="multibeam_blueview_p900_raster_standalone_macro"
+               params="name scale sonar_image_topic debug
+               sonar_image_raw_topic maxDistance raySkips plotScaler sensorGain writeLog
+               writeFrameInterval artificialVehicleVibration constantReflectivity
+               reflectivityDatabaseFile ray_visual">
+    <xacro:multibeam_sonar_standalone_link name="${name}"/>
+    <xacro:multibeam_blueview_p900_link name="${name}" scale="${scale}"/>
+    <joint name="multibeam_sonar_joint" type="fixed">
+      <parent link="${name}_standalone_base_link"/>
+      <child link="${name}_link"/>
+    </joint>
+    <xacro:multibeam_blueview_p900_raster_sensor name="${name}" sensor_link="${name}_link"
+                               sonar_image_topic="${sonar_image_topic}"  debug="${debug}"
+                               sonar_image_raw_topic="${sonar_image_raw_topic}"
+                               maxDistance="${maxDistance}" raySkips="${raySkips}"
+                               plotScaler="${plotScaler}" sensorGain="${sensorGain}"
+                               writeLog="${writeLog}" writeFrameInterval="${writeFrameInterval}"
+                               artificialVehicleVibration="${artificialVehicleVibration}"
+                               constantReflectivity="${constantReflectivity}"
+                               reflectivityDatabaseFile="${reflectivityDatabaseFile}"/>
+    <!-- Ray Visual -->
+    <xacro:multibeam_sonar_visual_link name="${name}"/>
+    <xacro:multibeam_sonar_visual_joint name="${name}"/>
+    <xacro:multibeam_blueview_p900_visual_ray name="${name}" ray_visual="${ray_visual}" />
   </xacro:macro>
   <xacro:macro name="multibeam_blueview_p900_ray_standalone_macro"
