Commit message: feature extraction

File: urdf/sensor/rexrov_sensors_main.xacro (robot description, xacro)
@@ -38,8 +38,8 @@
     <origin xyz="0 0 0" rpy="0 0 0"/>
   </xacro:default_imu_macro>
-  <!-- Mount cameras -->
+  <!-- Mount cameras <origin xyz="1.15 0.2 0.4" rpy="0 0.4 0"/>-->
   <xacro:include filename="$(find lias_ocean_sim)/urdf/sensor/camera/camera.xacro" />
-  <xacro:camera namespace="${namespace}" parent_link="${namespace}/base_link" suffix="right" update_rate="20" width="640" height="480">
-    <origin xyz="1.15 0.2 0.4" rpy="0 0.4 0"/>
+  <xacro:camera namespace="${namespace}" parent_link="${namespace}/base_link" suffix="right" update_rate="10" width="1024" height="768">
+    <origin xyz="1.2 0 -0.65" rpy="0 0 0"/>
   </xacro:camera>
   <!-- <xacro:camera namespace="${namespace}" parent_link="${namespace}/base_link" suffix="left" update_rate="24" width="640" height="360">
@@ -55,6 +55,26 @@
     inertial_reference_frame="${inertial_reference_frame}" />
   <!-- sonar -->
-  <!-- <xacro:include filename="$(find lias_ocean_sim)/urdf/sensor/sonar/multibeam_sonar_blueview_p900.xacro" />
-  <xacro:sonar_visualization_macro_no_blue_ray
+  <xacro:include filename="$(find lias_ocean_sim)/urdf/sensor/sonar/multibeam_sonar_blueview_p900.xacro" />
+<!--
+  <xacro:multibeam_blueview_p900_raster_macro
+    name="blueview_p900"
+    scale="1 1 1"
+    debug="false"
+    sonar_image_topic="sonar_image"
+    sonar_image_raw_topic="sonar_image_raw"
+    maxDistance="2"
+    raySkips="0"
+    plotScaler="0"
+    sensorGain="0.02"
+    writeLog="false"
+    writeFrameInterval="5"
+    artificialVehicleVibration="false"
+    constantReflectivity="false"
+    reflectivityDatabaseFile="variationalReflectivityDatabase.csv"
+    robot_link="${namespace}/base_link"
+    ray_visual="true">
+    <origin xyz="1.2 0.4 -0.65" rpy="0 0 0"/>
+  </xacro:multibeam_blueview_p900_raster_macro> -->
+  <xacro:multibeam_blueview_p900_ray_macro
     name="blueview_p900"
     scale="1 1 1"
@@ -63,8 +83,8 @@
     sonar_image_raw_topic="sonar_image_raw"
     robot_name="rexrov"
-    maxDistance="10"
+    maxDistance="5"
     raySkips="1"
-    plotScaler="0"
-    sensorGain="0.02"
+    sensorGain="0.1"
+    plotScaler="0.1"
     writeLog="false"
     writeFrameInterval="5"
@@ -74,25 +94,5 @@
     robot_link="${namespace}/base_link"
     ray_visual="true">
-    <origin xyz="1.2 0 -0.65" rpy="0 0 0"/>
-  </xacro:sonar_visualization_macro_no_blue_ray> -->
-  <!-- <xacro:sonar_visualization_macro
-    name="blueview_p900"
-    scale="1 1 1"
-    debug="false"
-    sonar_image_topic="sonar_image"
-    sonar_image_raw_topic="sonar_image_raw"
-    robot_name="rexrov"
-    maxDistance="10"
-    raySkips="1"
-    plotScaler="0"
-    sensorGain="0.02"
-    writeLog="false"
-    writeFrameInterval="5"
-    gaussian_noise_mean="0.0"
-    gaussian_noise_stddev="0.0"
-    fidelity="500"
-    robot_link="${namespace}/base_link"
-    ray_visual="true">
-    <origin xyz="1.2 0 -0.65" rpy="0 0 0"/>
-  </xacro:sonar_visualization_macro> -->
+    <origin xyz="1.2 0.5 -0.65" rpy="0 0 0"/>
+  </xacro:multibeam_blueview_p900_ray_macro>
 </robot>

File: urdf/sensor/sonar/multibeam_sonar_blueview_p900 copy.xacro (robot description, xacro)
@@ -65,4 +65,6 @@
           <!-- The CSV databsefile is located at the worlds folder -->
           <reflectivityDatabaseFile>${reflectivityDatabaseFile}</reflectivityDatabaseFile>
+          <customSDFTagReflectivity>true</customSDFTagReflectivity>
+          <customSDFTagDatabaseFile>customSDFTagDatabase.csv</customSDFTagDatabaseFile>
           <raySkips>${raySkips}</raySkips>
           <sensorGain>${sensorGain}</sensorGain>
@@ -242,5 +244,5 @@
                sonar_image_raw_topic maxDistance raySkips plotScaler sensorGain writeLog
                writeFrameInterval artificialVehicleVibration constantReflectivity
-               reflectivityDatabaseFile robot_link ray_visual">
+               reflectivityDatabaseFile robot_link ray_visual *origin">
     <xacro:multibeam_blueview_p900_link name="${name}" scale="${scale}"/>
     <joint name="multibeam_sonar_joint" type="fixed">

File: urdf/sensor/sonar/multibeam_sonar_blueview_p900_ray.xacro (robot description, xacro)
@@ -22,73 +22,4 @@
       </collision>
     </link>
-  </xacro:macro>
-  <!-- Generates a sensor element with Blueview P900 parameters -->
-  <xacro:macro name="multibeam_blueview_p900_raster_sensor"
-               params="name sensor_link sonar_image_topic sonar_image_raw_topic debug
-               maxDistance raySkips plotScaler sensorGain writeLog writeFrameInterval
-              artificialVehicleVibration constantReflectivity reflectivityDatabaseFile">
-    <gazebo reference="${sensor_link}">
-      <sensor name="${name}_sensor" type="depth">
-        <visualize>true</visualize>
-        <always_on>true</always_on>
-        <update_rate>10</update_rate>
-        <camera>
-          <!-- 60 degrees for the oculus-m1200d at 2.1MHz mode -->
-          <horizontal_fov>1.0471975512</horizontal_fov>
-          <image>
-            <width>256</width>
-            <!-- Set vertical FOV by setting image height -->
-            <!-- Approx 2 times the spec sheet (sepc: 12 deg.) -->
-            <height>102</height>
-            <format>R8G8B8</format>
-          </image>
-          <clip>
-            <near>0.1</near>            <!-- optimal 2m-60m -->
-            <far>5</far>
-          </clip>
-          <depth_camera>
-            <output>depths</output>
-          </depth_camera>
-          <save enabled="false">
-            <path>/tmp/camera</path>
-          </save>
-        </camera>
-        <plugin filename="libnps_multibeam_sonar_ros_plugin.so" name="${name}_sensor_controller">
-          <!-- Sonar properties -->
-         <verticalFOV>20</verticalFOV>
-          <sonarFreq>2100e3</sonarFreq>
-          <bandwidth>265.5e3</bandwidth>
-          <soundSpeed>1500</soundSpeed>
-          <sourceLevel>150</sourceLevel>
-          <maxDistance>3</maxDistance>
-          <!-- custom SDF Tag works when constantReflectivity is false -->
-          <constantReflectivity>false</constantReflectivity>
-          <customSDFTagReflectivity>false</customSDFTagReflectivity>
-          <!-- The CSV databsefile is located at the worlds folder -->
-          <customSDFTagDatabaseFile>customSDFTagDatabase.csv</customSDFTagDatabaseFile>
-          <!-- reflectivity database (by model name) works -->
-          <!-- when both constantReflectivity and customSDFTagReflectivity are false -->
-          <reflectivityDatabaseFile>variationalReflectivityDatabase.csv</reflectivityDatabaseFile>
-          <raySkips>1</raySkips>
-          <sensorGain>1</sensorGain>
-          <plotScaler>0</plotScaler>
-          <writeLog>false</writeLog>
-          <debugFlag>true</debugFlag>
-          <writeFrameInterval>5</writeFrameInterval>
-          <artificialVehicleVibration>${artificialVehicleVibration}</artificialVehicleVibration>
-          <!-- This name is prepended to ROS topics -->
-          <cameraName>${name}</cameraName>
-          <!-- ROS publication topics -->
-          <imageTopicName>${name}/image_raw</imageTopicName>
-          <cameraInfoTopicName>${name}/image_raw/camera_info</cameraInfoTopicName>
-          <pointCloudTopicName>${name}/point_cloud</pointCloudTopicName>
-          <depthImageTopicName>${name}/image_depth</depthImageTopicName>
-          <depthImageCameraInfoTopicName>${name}/image_depth/camera_info</depthImageCameraInfoTopicName>
-          <sonarImageRawTopicName>${sonar_image_raw_topic}</sonarImageRawTopicName>
-          <sonarImageTopicName>${sonar_image_topic}</sonarImageTopicName>
-          <frameName>${name}_forward_sonar_optical_link</frameName>
-        </plugin>
-      </sensor>
-    </gazebo>
   </xacro:macro>
   <xacro:macro name="multibeam_blueview_p900_ray_sensor"
@@ -104,25 +35,25 @@
           <scan>
             <!-- Set horizontal FOV by setting image height -->
-            <!-- 512 beams with 90 degrees horizontal FOV (M900-90) -->
+            <!-- 512 beams with 40 degrees horizontal FOV (M900-90) -->
             <horizontal>
-              <samples>768</samples>
+              <samples>512</samples>
               <resolution>1</resolution>
               <min_angle>-0.52</min_angle>
               <max_angle>0.52</max_angle>
             </horizontal>
-            <!-- Set vertical FOV by setting image height -->
+            <!-- Set vertical FOV 20 degree by setting image height -->
             <!-- Approx 2 times the spec sheet (sepc: 20 deg.) -->
             <vertical>
-              <samples>96</samples>
-              <resolution>1</resolution>
-              <min_angle>-0.26</min_angle>
-              <max_angle>0.26</max_angle>
+              <samples>256</samples>
+              <resolution>1</resolution>
+              <min_angle>-0.175</min_angle>
+              <max_angle>0.175</max_angle>
             </vertical>
           </scan>
           <range>
             <!-- min range is a collision range no need to change-->
-            <min>1.5</min>
-            <max>${maxDistance + 2}</max>
-            <resolution>1</resolution>
+            <min>0.1</min>
+            <max>5</max>
+            <resolution>0.1</resolution>
           </range>
           <noise>
@@ -132,6 +63,6 @@
                 stddev of 0.01m will put 99.7% of samples within 0.03m of the true
                 reading. -->
-            <mean>${gaussian_noise_mean}</mean>
-            <stddev>${gaussian_noise_stddev}</stddev>
+            <mean>0</mean>
+            <stddev>0</stddev>
           </noise>
         </ray>
@@ -145,16 +76,10 @@
         <plugin filename="libnps_multibeam_sonar_ray_ros_plugin.so" name="${name}_sensor_controller">
           <!-- Sonar properties -->
-          <verticalFOV>30</verticalFOV>
-          <sonarFreq>100e4</sonarFreq>
-          <bandwidth>15e4</bandwidth>
+          <verticalFOV>20</verticalFOV>
+          <sonarFreq>900e3</sonarFreq>
+          <bandwidth>29.9e3</bandwidth>
           <soundSpeed>1500</soundSpeed>
-          <sourceLevel>185</sourceLevel>
+          <sourceLevel>220</sourceLevel>
           <maxDistance>${maxDistance}</maxDistance>
-          <!-- <verticalFOV>20</verticalFOV>
-          <sonarFreq>2100e3</sonarFreq>
-          <bandwidth>265.5e3</bandwidth>
-          <soundSpeed>1500</soundSpeed>
-          <sourceLevel>150</sourceLevel>
-          <maxDistance>5</maxDistance> -->
           <raySkips>${raySkips}</raySkips>
           <sensorGain>${sensorGain}</sensorGain>
@@ -204,6 +129,6 @@
               <samples>100</samples>
               <resolution>1</resolution>
-              <min_angle>-0.785398</min_angle>
-              <max_angle>0.785398</max_angle>
+              <min_angle>-0.52</min_angle>
+              <max_angle>0.52</max_angle>
             </horizontal>
             <vertical>
@@ -224,5 +149,5 @@
   </xacro:macro>
   <xacro:arg name="standalone" default="false"/>
-  <xacro:arg name="gpu_ray" default="false"/>
+  <xacro:arg name="gpu_ray" default="true"/>
   <xacro:arg name="name" default="blueview_p900"/>
   <xacro:arg name="maxDistance" default="10"/>
@@ -242,5 +167,5 @@
   <xacro:arg name="gaussian_noise_mean" default="0.0"/>
   <xacro:arg name="gaussian_noise_stddev" default="0.0"/>
-  <xacro:arg name="fidelity" default="500"/>
+  <xacro:arg name="fidelity" default="64"/>
   <xacro:arg name="robot_name" default=""/>
   <!-- Top level macro for generating the link, sensor, joint combo
@@ -249,29 +174,4 @@
        but sensor orientation will always be forward and down relative to
        the robot link (robot_link parameter). -->
-  <xacro:macro name="multibeam_blueview_p900_raster_macro"
-               params="name scale sonar_image_topic debug
-               sonar_image_raw_topic maxDistance raySkips plotScaler sensorGain writeLog
-               writeFrameInterval artificialVehicleVibration constantReflectivity
-               reflectivityDatabaseFile robot_link ray_visual *origin">
-    <xacro:multibeam_blueview_p900_link name="${name}" scale="${scale}"/>
-    <joint name="multibeam_sonar_joint" type="fixed">
-      <parent link="${robot_link}"/>
-      <child link="${name}_link"/>
-      <xacro:insert_block name="origin"/>\
-    </joint>
-    <xacro:multibeam_blueview_p900_raster_sensor name="${name}" debug="${debug}"
-                               sonar_image_topic="${sonar_image_topic}"  sensor_link="${name}_link"
-                               sonar_image_raw_topic="${sonar_image_raw_topic}"
-                               maxDistance="${maxDistance}" raySkips="${raySkips}"
-                               plotScaler="${plotScaler}" sensorGain="${sensorGain}"
-                               writeLog="${writeLog}" writeFrameInterval="${writeFrameInterval}"
-                               artificialVehicleVibration="${artificialVehicleVibration}"
-                               constantReflectivity="${constantReflectivity}"
-                               reflectivityDatabaseFile="${reflectivityDatabaseFile}"/>
-    <!-- Ray Visual -->
-    <xacro:multibeam_sonar_visual_link name="${name}"/>
-    <xacro:multibeam_sonar_visual_joint name="${name}"/>
-    <xacro:multibeam_blueview_p900_visual_ray name="${name}" ray_visual="${ray_visual}"/>
-  </xacro:macro>
   <xacro:macro name="multibeam_blueview_p900_ray_macro"
                params="name scale debug sonar_image_topic sonar_image_raw_topic
@@ -300,9 +200,9 @@
     <xacro:multibeam_blueview_p900_visual_ray name="${name}" ray_visual="${ray_visual}"/>
   </xacro:macro>
-  <xacro:macro name="multibeam_blueview_p900_macro"
-               params="name scale sonar_image_topic debug gpu_ray robot_name
-               sonar_image_raw_topic maxDistance raySkips plotScaler sensorGain writeLog
+  <xacro:macro name="sonar_visualization_macro"
+               params="name scale debug sonar_image_topic sonar_image_raw_topic
+               robot_name
+               maxDistance raySkips plotScaler sensorGain writeLog
                writeFrameInterval gaussian_noise_mean gaussian_noise_stddev fidelity
-               artificialVehicleVibration constantReflectivity reflectivityDatabaseFile
                robot_link ray_visual *origin">
     <xacro:multibeam_blueview_p900_link name="${name}" scale="${scale}"/>
@@ -310,32 +210,23 @@
       <parent link="${robot_link}"/>
       <child link="${name}_link"/>
-      <xacro:insert_block name="origin"/>
-    </joint>
-    <xacro:if value="$(arg gpu_ray)">
-      <xacro:multibeam_blueview_p900_ray_sensor name="${name}" sensor_link="${name}_link"
-                                sonar_image_topic="${sonar_image_topic}" debug="${debug}"
-                                sonar_image_raw_topic="${sonar_image_raw_topic}"
-                                maxDistance="${maxDistance}" raySkips="${raySkips}"
-                                plotScaler="${plotScaler}" sensorGain="${sensorGain}"
-                                writeLog="${writeLog}" writeFrameInterval="${writeFrameInterval}"
-                                gaussian_noise_mean="${gaussian_noise_mean}"
-                                gaussian_noise_stddev="${gaussian_noise_stddev}"
-                                fidelity="${fidelity}" pcl_topic_name="${robot_name}/${name}_point_cloud"/>
-    </xacro:if>
-    <xacro:unless value="$(arg gpu_ray)">
-      <xacro:multibeam_blueview_p900_raster_sensor name="${name}" debug="${debug}"
-                                sonar_image_topic="${sonar_image_topic}"  sensor_link="${name}_link"
-                                sonar_image_raw_topic="${sonar_image_raw_topic}"
-                                maxDistance="${maxDistance}" raySkips="${raySkips}"
-                                plotScaler="${plotScaler}" sensorGain="${sensorGain}"
-                                writeLog="${writeLog}" writeFrameInterval="${writeFrameInterval}"
-                                artificialVehicleVibration="${artificialVehicleVibration}"
-                                constantReflectivity="${constantReflectivity}"
-                                reflectivityDatabaseFile="${reflectivityDatabaseFile}"/>
-    </xacro:unless>
+      <xacro:insert_block name="origin"/>\
+    </joint>
     <!-- Ray Visual -->
     <xacro:multibeam_sonar_visual_link name="${name}"/>
     <xacro:multibeam_sonar_visual_joint name="${name}"/>
     <xacro:multibeam_blueview_p900_visual_ray name="${name}" ray_visual="${ray_visual}"/>
+  </xacro:macro>
+  <xacro:macro name="sonar_visualization_macro_no_blue_ray"
+               params="name scale debug sonar_image_topic sonar_image_raw_topic
+               robot_name
+               maxDistance raySkips plotScaler sensorGain writeLog
+               writeFrameInterval gaussian_noise_mean gaussian_noise_stddev fidelity
+               robot_link ray_visual *origin">
+    <xacro:multibeam_blueview_p900_link name="${name}" scale="${scale}"/>
+    <joint name="multibeam_sonar_joint" type="fixed">
+      <parent link="${robot_link}"/>
+      <child link="${name}_link"/>
+      <xacro:insert_block name="origin"/>\
+    </joint>
   </xacro:macro>
   <!-- For standalone -->
@@ -345,29 +236,4 @@
       <static>true</static>
     </gazebo>
-  </xacro:macro>
-  <xacro:macro name="multibeam_blueview_p900_raster_standalone_macro"
-               params="name scale sonar_image_topic debug
-               sonar_image_raw_topic maxDistance raySkips plotScaler sensorGain writeLog
-               writeFrameInterval artificialVehicleVibration constantReflectivity
-               reflectivityDatabaseFile ray_visual">
-    <xacro:multibeam_sonar_standalone_link name="${name}"/>
-    <xacro:multibeam_blueview_p900_link name="${name}" scale="${scale}"/>
-    <joint name="multibeam_sonar_joint" type="fixed">
-      <parent link="${name}_standalone_base_link"/>
-      <child link="${name}_link"/>
-    </joint>
-    <xacro:multibeam_blueview_p900_raster_sensor name="${name}" sensor_link="${name}_link"
-                               sonar_image_topic="${sonar_image_topic}"  debug="${debug}"
-                               sonar_image_raw_topic="${sonar_image_raw_topic}"
-                               maxDistance="${maxDistance}" raySkips="${raySkips}"
-                               plotScaler="${plotScaler}" sensorGain="${sensorGain}"
-                               writeLog="${writeLog}" writeFrameInterval="${writeFrameInterval}"
-                               artificialVehicleVibration="${artificialVehicleVibration}"
-                               constantReflectivity="${constantReflectivity}"
-                               reflectivityDatabaseFile="${reflectivityDatabaseFile}"/>
-    <!-- Ray Visual -->
-    <xacro:multibeam_sonar_visual_link name="${name}"/>
-    <xacro:multibeam_sonar_visual_joint name="${name}"/>
-    <xacro:multibeam_blueview_p900_visual_ray name="${name}" ray_visual="${ray_visual}" />
   </xacro:macro>
   <xacro:macro name="multibeam_blueview_p900_ray_standalone_macro"
